Commit message: ur5 perfect urdf with old end effector 6 points movement

File: src/leaf_robot_description/urdf/demo_leaf.urdf (robot description, URDF)
Before this commit: robot leaf_robot_description, 8 links, 7 joints
Links:
- added link big_section_1; collision cylinder length=0.2 radius=0.30; visual cylinder length=0.2 radius=0.30
- added link big_section_2; collision cylinder length=0.2 radius=0.30; visual cylinder length=0.2 radius=0.30
- added link big_section_3; collision cylinder length=0.2 radius=0.30; visual cylinder length=0.2 radius=0.30
- added link big_section_4; collision cylinder length=0.2 radius=0.30; visual cylinder length=0.2 radius=0.30
- added link big_section_5; collision cylinder length=0.2 radius=0.30; visual cylinder length=0.2 radius=0.30
- added link big_section_6; collision cylinder length=0.2 radius=0.30; visual cylinder length=0.2 radius=0.30
- added link big_section_7; collision cylinder length=0.2 radius=0.30; visual cylinder length=0.2 radius=0.30
- added link big_section_8; collision cylinder length=0.2 radius=0.30; visual cylinder length=0.2 radius=0.30
- added link gripper_base_link; visual box size=0.02 0.06 0.02
- added link left_finger; visual box size=0.02 0.01 0.235
- added link right_finger; visual box size=0.02 0.01 0.235
- added link small_cylinder_1; collision cylinder length=1.6 radius=0.015; visual cylinder length=1.6 radius=0.015
- link J_6: mass 0.14576 -> None; geometry collision box size=0.04 0.02 0.02; visual cylinder length=0.1 radius=0.03
Joints:
- added joint Gripper: type fixed, parent J_6, child gripper_base_link, origin xyz=0 -0.06 0 rpy=1.5708 0 0
- added joint big_section_1_joint: type fixed, parent base_footprint, child big_section_1, origin xyz=0.30 -0.45 0.1 rpy=0 0 0
- added joint big_section_2_joint: type fixed, parent base_footprint, child big_section_2, origin xyz=0.30 -0.45 0.3 rpy=0 0 0
- added joint big_section_3_joint: type fixed, parent base_footprint, child big_section_3, origin xyz=0.30 -0.45 0.5 rpy=0 0 0
- added joint big_section_4_joint: type fixed, parent base_footprint, child big_section_4, origin xyz=0.30 -0.45 0.7 rpy=0 0 0
- added joint big_section_5_joint: type fixed, parent base_footprint, child big_section_5, origin xyz=0.30 -0.45 0.9 rpy=0 0 0
- added joint big_section_6_joint: type fixed, parent base_footprint, child big_section_6, origin xyz=0.30 -0.45 1.1 rpy=0 0 0
- added joint big_section_7_joint: type fixed, parent base_footprint, child big_section_7, origin xyz=0.30 -0.45 1.3 rpy=0 0 0
- added joint big_section_8_joint: type fixed, parent base_footprint, child big_section_8, origin xyz=0.30 -0.45 1.5 rpy=0 0 0
- added joint left_finger_joint: type prismatic, parent gripper_base_link, child left_finger, origin xyz=0 0.025 0, axis 0 -1 0, limit lower=0.0 upper=0.02 effort=10 velocity=0.1
- added joint right_finger_joint: type prismatic, parent gripper_base_link, child right_finger, origin xyz=0 -0.025 0, axis 0 -1 0, limit lower=0.0 upper=0.02 effort=10 velocity=0.1, mimic joint=left_finger_joint multiplier=-1.0
- added joint small_cylinder_1_joint: type fixed, parent base_footprint, child small_cylinder_1, origin xyz=0.30 -0.45 0.8 rpy=0 0 0
- joint ROT_3: axis 0 0 1 -> 0 1 0; limit lower=-3.14 upper=3.14 effort=10 velocity=1.0 -> lower=-6.28 upper=6.28 effort=50 velocity=1.0; origin xyz=-0.00088397 -0.0023385 -0.0725 rpy=1.5708 -0.70269 2.7802 -> xyz=-0.0015905 -0.0042271 -0.078525 rpy=0 0 -0.353599
