Commit message: ur5 with green colour custom gripper with working 6 points

File: src/leaf_robot_description/urdf/leaf_robot.urdf (robot description, URDF)
Before this commit: robot leaf_robot_description, 8 links, 7 joints
Links:
- added link gripper_base_link; visual box size=0.02 0.06 0.02
- added link left_finger; visual box size=0.02 0.01 0.235
- added link right_finger; visual box size=0.02 0.01 0.235
- link J_6: mass 0.14576 -> None; geometry collision box size=0.04 0.02 0.02; visual cylinder length=0.1 radius=0.03
Joints:
- added joint Gripper: type fixed, parent J_6, child gripper_base_link, origin xyz=0 -0.06 0 rpy=1.5708 0 0
- added joint left_finger_joint: type prismatic, parent gripper_base_link, child left_finger, origin xyz=0 0.025 0, axis 0 -1 0, limit lower=0.0 upper=0.02 effort=10 velocity=0.1
- added joint right_finger_joint: type prismatic, parent gripper_base_link, child right_finger, origin xyz=0 -0.025 0, axis 0 -1 0, limit lower=0.0 upper=0.02 effort=10 velocity=0.1, mimic joint=left_finger_joint multiplier=-1.0
- joint ROT_3: axis 0 0 1 -> 0 1 0; limit lower=-3.14 upper=3.14 effort=10 velocity=1.0 -> lower=-6.28 upper=6.28 effort=50 velocity=1.0; origin xyz=-0.00088397 -0.0023385 -0.0725 rpy=1.5708 -0.70269 2.7802 -> xyz=-0.0015905 -0.0042271 -0.078525 rpy=0 0 -0.353599

File: src/leaf_robot_moveit_config/config/leaf_robot_description.ros2_control.xacro (robot description, xacro)
@@ -13,5 +13,4 @@
                   <param name="initial_value">${initial_positions['ROT_1']}</param>
                 </state_interface>
-                <state_interface name="velocity"/>
             </joint>
             <joint name="PITCH_1">
@@ -20,5 +19,4 @@
                   <param name="initial_value">${initial_positions['PITCH_1']}</param>
                 </state_interface>
-                <state_interface name="velocity"/>
             </joint>
             <joint name="PITCH_2">
@@ -27,5 +25,4 @@
                   <param name="initial_value">${initial_positions['PITCH_2']}</param>
                 </state_interface>
-                <state_interface name="velocity"/>
             </joint>
             <joint name="PITCH_3">
@@ -34,5 +31,4 @@
                   <param name="initial_value">${initial_positions['PITCH_3']}</param>
                 </state_interface>
-                <state_interface name="velocity"/>
             </joint>
             <joint name="ROT_2">
@@ -41,5 +37,4 @@
                   <param name="initial_value">${initial_positions['ROT_2']}</param>
                 </state_interface>
-                <state_interface name="velocity"/>
             </joint>
             <joint name="ROT_3">
@@ -48,5 +43,10 @@
                   <param name="initial_value">${initial_positions['ROT_3']}</param>
                 </state_interface>
-                <state_interface name="velocity"/>
+            </joint>
+            <joint name="left_finger_joint">
+                <command_interface name="position"/>
+                <state_interface name="position">
+                  <param name="initial_value">${initial_positions['left_finger_joint']}</param>
+                </state_interface>
             </joint>
         </ros2_control>

Commit message: ur5 with origin at gripper with ik

File: src/leaf_robot_description/urdf/leaf_robot.urdf (robot description, URDF)
Before this commit: robot leaf_robot_description, 11 links, 10 joints
Links:
- added link link_tcp; collision sphere radius=0.005; visual sphere radius=0.008
- link right_finger: geometry collision box size=0.02 0.01 0.235; visual box size=0.02 0.01 0.235
Joints:
- added joint tcp_joint: type fixed, parent gripper_base_link, child link_tcp, origin xyz=0 0 0.17625 rpy=0 0 0

File: src/leaf_robot_moveit_config/config/leaf_robot_description.ros2_control.xacro (robot description, xacro)
@@ -13,4 +13,5 @@
                   <param name="initial_value">${initial_positions['ROT_1']}</param>
                 </state_interface>
+                <state_interface name="velocity"/>
             </joint>
             <joint name="PITCH_1">
@@ -19,4 +20,5 @@
                   <param name="initial_value">${initial_positions['PITCH_1']}</param>
                 </state_interface>
+                <state_interface name="velocity"/>
             </joint>
             <joint name="PITCH_2">
@@ -25,4 +27,5 @@
                   <param name="initial_value">${initial_positions['PITCH_2']}</param>
                 </state_interface>
+                <state_interface name="velocity"/>
             </joint>
             <joint name="PITCH_3">
@@ -31,4 +34,5 @@
                   <param name="initial_value">${initial_positions['PITCH_3']}</param>
                 </state_interface>
+                <state_interface name="velocity"/>
             </joint>
             <joint name="ROT_2">
@@ -37,4 +41,5 @@
                   <param name="initial_value">${initial_positions['ROT_2']}</param>
                 </state_interface>
+                <state_interface name="velocity"/>
             </joint>
             <joint name="ROT_3">
@@ -43,4 +48,5 @@
                   <param name="initial_value">${initial_positions['ROT_3']}</param>
                 </state_interface>
+                <state_interface name="velocity"/>
             </joint>
             <joint name="left_finger_joint">
@@ -49,4 +55,5 @@
                   <param name="initial_value">${initial_positions['left_finger_joint']}</param>
                 </state_interface>
+                <state_interface name="velocity"/>
             </joint>
         </ros2_control>
